File: ergogen/pcb/board.kicad_pcb (KiCad board)
At the start: 2 copper layers, 151 x 112.4 mm, 53 parts

Commit message: journal: 02/06/2025
Other:
- board text added: "Made By: Ankush Roy Started: 25th May 2025 Event: Highway Keyboard Name: SplitWave"
