File: pcb/board.kicad_pcb (KiCad board)
At the start: 2 copper layers, 151 x 112.4 mm, 53 parts

Commit message: journal: 05/06/2025
Parts:
- moved B1 0.97 mm to (224.4, 99.6)
- moved T1 0.72 mm to (225.1, 89.9)
Routing:
- net RST: track 68.2 -> 79.6 mm
- net GND: track 127.9 -> 117.2 mm
